Commit message: move urdf to spotmicro_description package

File: src/spotmicro_description/urdf/spotmicro.urdf.xacro (robot description, xacro)
@@ -35,5 +35,5 @@
         <xacro:if value="${left}">
         <geometry>
-          <mesh filename="package://spotmicro_rviz/urdf/stl/lshoulder.stl" scale="0.001 0.001 0.001"/>
+          <mesh filename="package://spotmicro_description/urdf/stl/lshoulder.stl" scale="0.001 0.001 0.001"/>
         </geometry>
         <origin rpy="0 0 3.14159" xyz="0.135 0.015 -0.01"/>
@@ -41,5 +41,5 @@
         <xacro:unless value="${left}">
         <geometry>
-          <mesh filename="package://spotmicro_rviz/urdf/stl/rshoulder.stl" scale="0.001 0.001 0.001"/>
+          <mesh filename="package://spotmicro_description/urdf/stl/rshoulder.stl" scale="0.001 0.001 0.001"/>
         </geometry>
         <origin rpy="0 0 3.14159" xyz="0.135 0.095 -0.01"/>
@@ -74,5 +74,5 @@
         <xacro:if value="${left}">
         <geometry>
-          <mesh filename="package://spotmicro_rviz/urdf/stl/larm_cover.stl" scale="0.001 0.001 0.001"/>
+          <mesh filename="package://spotmicro_description/urdf/stl/larm_cover.stl" scale="0.001 0.001 0.001"/>
         </geometry>
         <origin rpy="0 -0.139 3.14159" xyz="0.130 -0.040 -0.025"/>
@@ -80,5 +80,5 @@
         <xacro:unless value="${left}">
         <geometry>
-          <mesh filename="package://spotmicro_rviz/urdf/stl/rarm_cover.stl" scale="0.001 0.001 0.001"/>
+          <mesh filename="package://spotmicro_description/urdf/stl/rarm_cover.stl" scale="0.001 0.001 0.001"/>
         </geometry>
         <origin rpy="0 -0.139 3.14159" xyz="0.130 0.15 -0.025"/>
@@ -91,5 +91,5 @@
         <xacro:if value="${left}">
         <geometry>
-          <mesh filename="package://spotmicro_rviz/urdf/stl/larm.stl" scale="0.001 0.001 0.001"/>
+          <mesh filename="package://spotmicro_description/urdf/stl/larm.stl" scale="0.001 0.001 0.001"/>
         </geometry>
         <origin rpy="0 -0.139 3.14159" xyz="0.130 -0.040 -0.025"/>
@@ -97,5 +97,5 @@
         <xacro:unless value="${left}">
         <geometry>
-          <mesh filename="package://spotmicro_rviz/urdf/stl/rarm.stl" scale="0.001 0.001 0.001"/>
+          <mesh filename="package://spotmicro_description/urdf/stl/rarm.stl" scale="0.001 0.001 0.001"/>
         </geometry>
         <origin rpy="0 -0.139 3.14159" xyz="0.130 0.15 -0.025"/>
@@ -140,5 +140,5 @@
         <xacro:if value="${left}">
         <geometry>
-          <mesh filename="package://spotmicro_rviz/urdf/stl/lfoot.stl" scale="0.001 0.001 0.001"/>
+          <mesh filename="package://spotmicro_description/urdf/stl/lfoot.stl" scale="0.001 0.001 0.001"/>
         </geometry>
         <origin rpy="0 0 3.14159" xyz="0.120 -0.04 0.1"/>
@@ -146,5 +146,5 @@
         <xacro:unless value="${left}">
         <geometry>
-          <mesh filename="package://spotmicro_rviz/urdf/stl/rfoot.stl" scale="0.001 0.001 0.001"/>
+          <mesh filename="package://spotmicro_description/urdf/stl/rfoot.stl" scale="0.001 0.001 0.001"/>
         </geometry>
         <origin rpy="0 0 3.14159" xyz="0.120 0.15 0.1"/>
@@ -178,5 +178,5 @@
       <visual>
         <geometry>
-        <mesh filename="package://spotmicro_rviz/urdf/stl/foot.stl" scale="0.001 0.001 0.001"/>
+        <mesh filename="package://spotmicro_description/urdf/stl/foot.stl" scale="0.001 0.001 0.001"/>
         </geometry>
         <origin rpy="0 -0.40010 3.14159" xyz="0.00 0.01 0.015"/>
@@ -217,5 +217,5 @@
     <visual>
       <geometry>
-        <mesh filename="package://spotmicro_rviz/urdf/stl/mainbody.stl" scale="0.001 0.001 0.001"/>
+        <mesh filename="package://spotmicro_description/urdf/stl/mainbody.stl" scale="0.001 0.001 0.001"/>
       </geometry>
       <material name="black"/>
@@ -237,5 +237,5 @@
     <visual>
       <geometry>
-        <mesh filename="package://spotmicro_rviz/urdf/stl/rplidar_main.STL" scale="0.001 0.001 0.001"/>
+        <mesh filename="package://spotmicro_description/urdf/stl/rplidar_main.STL" scale="0.001 0.001 0.001"/>
       </geometry>
       <material name="black"/>
@@ -261,5 +261,5 @@
     <visual>
       <geometry>
-        <mesh filename="package://spotmicro_rviz/urdf/stl/backpart.stl" scale="0.001 0.001 0.001"/>
+        <mesh filename="package://spotmicro_description/urdf/stl/backpart.stl" scale="0.001 0.001 0.001"/>
       </geometry>
       <origin rpy="0 0 3.14159" xyz="0.04 0.055 -0.010"/>
@@ -284,5 +284,5 @@
     <visual>
       <geometry>
-        <mesh filename="package://spotmicro_rviz/urdf/stl/frontpart.stl" scale="0.001 0.001 0.001"/>
+        <mesh filename="package://spotmicro_description/urdf/stl/frontpart.stl" scale="0.001 0.001 0.001"/>
       </geometry>
       <origin rpy="0 0 3.14159" xyz="0.040 0.055 -0.010"/>
